File: Schematic/Test_board/SD card/SD Card/SD Card.sch (KiCad schematic (older format))
At the start: 10 parts, among them J1 Conn_01x07_Female, J3 Conn_01x05_Female, J4 503398-1892, U2 ICM-20602, U3 TXB0104PW

Commit message: Added power distribution to test board.
Added the schematic and footprints needed for power distribution in test board.

2.2. Basic Sensor Suite
Parts:
- added C5: 15uF, Capacitor_SMD:C_1812_4532Metric_Pad1.57x3.40mm_HandSolder, symbol Device:C
- added C6: 0.01uF, Capacitor_SMD:C_1206_3216Metric_Pad1.33x1.80mm_HandSolder, symbol Device:C
- added C7, C8: 0.1uF, Capacitor_SMD:C_1206_3216Metric_Pad1.33x1.80mm_HandSolder, symbol Device:C
- added C9: 1uF, Capacitor_SMD:C_1812_4532Metric_Pad1.57x3.40mm_HandSolder, symbol Device:C
- added D1: D, Diode_SMD:D_SMA_Handsoldering, symbol Device:D
- added D2: D_Bridge_+AA-, TTS_UART:KBP306GTB, symbol Device:D_Bridge_+AA-
- added J2: Conn_01x02_Female, Connector_PinHeader_2.54mm:PinHeader_1x02_P2.54mm_Vertical, symbol Connector:Conn_01x02_Female
- added J5: Screw_Terminal_01x02, TerminalBlock_Phoenix:TerminalBlock_Phoenix_PT-1,5-2-5.0-H_1x02_P5.00mm_Horizontal, symbol Connector:Screw_Terminal_01x02
- added L1: 100uH, Inductor_SMD:L_TDK_SLF7045, symbol Device:L
- added R1: 1, Resistor_SMD:R_1206_3216Metric_Pad1.30x1.75mm_HandSolder, symbol Device:R
- added R3: 3.01k, Resistor_SMD:R_1206_3216Metric_Pad1.30x1.75mm_HandSolder, symbol Device:R
- added R4: 1k, Resistor_SMD:R_1206_3216Metric_Pad1.30x1.75mm_HandSolder, symbol Device:R
- added R5: 100k, Resistor_SMD:R_1206_3216Metric_Pad1.30x1.75mm_HandSolder, symbol Device:R
- added R6: 200k, Resistor_SMD:R_1206_3216Metric_Pad1.30x1.75mm_HandSolder, symbol Device:R
- added U1: LM25007MM_NOPB, LM25007MM:LM25007MM&slash_NOPB, symbol SD-Card-rescue:LM25007MM_NOPB-lm25007-SD-Card-rescue
- J4: symbol uSD_card:503398-1892 -> SD-Card-rescue:503398-1892-uSD_card-SD-Card-rescue
Connections:
- net labels added: BST, FB, RON
- wire segments 65 -> 121

Commit message: Test board PCB design
Board includes SD card, IMU and PDU

2.2 Basic Sensor Suite
Parts:
- removed J1: Conn_01x07_Female, Connector_PinHeader_2.54mm:PinHeader_1x07_P2.54mm_Vertical, symbol Connector:Conn_01x07_Female
- added J1: Conn_01x06_Female, Connector_PinHeader_2.54mm:PinHeader_1x06_P2.54mm_Vertical, symbol Connector:Conn_01x06_Female
- J4: symbol SD-Card-rescue:503398-1892-uSD_card-SD-Card-rescue -> SD-Card-rescue:503398-1892-uSD_card-SD-Card-rescue-SD-Card-rescue
- U1: symbol SD-Card-rescue:LM25007MM_NOPB-lm25007-SD-Card-rescue -> SD-Card-rescue:LM25007MM_NOPB-lm25007-SD-Card-rescue-SD-Card-rescue
Connections:
- net 3.3V: now also J1.2 (Pin_2)
- net 5v: now also J1.1 (Pin_1)
- net at U3.10 (B4): now also J1.6 (Pin_6)
- net at U3.11 (B3): now also J1.5 (Pin_5)
- net at U3.12 (B2): now also J1.4 (Pin_4)
- net at U3.13 (B1): now also J1.3 (Pin_3)
Changed lines of the file:
@@
 	4100 2050 3550 2050
-$Comp
-L power:GND #PWR0102
-U 1 1 5FDFE3F5
-P 4450 2050
-F 0 "#PWR0102" H 4450 1800 50  0001 C CNN
-F 1 "GND" H 4455 1877 50  0000 C CNN
-F 2 "" H 4450 2050 50  0001 C CNN
-F 3 "" H 4450 2050 50  0001 C CNN
-	1    4450 2050
-	1    0    0    -1
-$EndComp
-Wire Wire Line
-	4450 2050 4450 2000
 $Comp
 L power:GND #PWR0103
@@
 	4200 1800 4650 1800
 Wire Wire Line
-	4450 2000 4650 2000
-Wire Wire Line
 	4100 1900 4650 1900
 Text Label 4650 1400 2    50   ~ 0
@@
 	3250 1050 3250 900
 $Comp
-L SD-Card-rescue:503398-1892-uSD_card-SD-Card-rescue J4
+L SD-Card-rescue:503398-1892-uSD_card-SD-Card-rescue-SD-Card-rescue J4
 U 1 1 5FDB0DED
 P 1400 1650
@@
 	2300 2250 2300 2150
 $Comp
-L Connector:Conn_01x07_Female J1
-U 1 1 5FE6E166
-P 4850 1700
-F 0 "J1" H 4878 1726 50  0000 L CNN
-F 1 "Conn_01x07_Female" H 4878 1635 50  0000 L CNN
-F 2 "Connector_PinHeader_2.54mm:PinHeader_1x07_P2.54mm_Vertical" H 4850 1700 50  0001 C CNN
-F 3 "~" H 4850 1700 50  0001 C CNN
-	1    4850 1700
-	1    0    0    -1
-$EndComp
-$Comp
 L Device:D D1
 U 1 1 5FDBDAD8
@@
 $EndComp
 $Comp
-L SD-Card-rescue:LM25007MM_NOPB-lm25007-SD-Card-rescue U1
+L SD-Card-rescue:LM25007MM_NOPB-lm25007-SD-Card-rescue-SD-Card-rescue U1
 U 1 1 5FE77355
 P 7100 4050
@@
 	1    0    0    -1
 $EndComp
+$Comp
+L Connector:Conn_01x06_Female J1
+U 1 1 5FDCE218
+P 4850 1600
+F 0 "J1" H 4878 1576 50  0000 L CNN
+F 1 "Conn_01x06_Female" H 4878 1485 50  0000 L CNN
+F 2 "Connector_PinHeader_2.54mm:PinHeader_1x06_P2.54mm_Vertical" H 4850 1600 50  0001 C CNN
+F 3 "~" H 4850 1600 50  0001 C CNN
+	1    4850 1600
+	1    0    0    -1
+$EndComp
