File: Schematic/Mega_Shield/Mega_Shield.sch (KiCad schematic (older format))
At the start: 24 parts, among them J1 Mini-DIN-4, J10 Conn_01x08, J11 Conn_01x08, J12 Conn_02x18_Odd_Even, J13 Conn_01x08, J14 Conn_01x08, J15 Conn_01x08, J16 Conn_01x10, J2 Mini-DIN-4, J3 Mini-DIN-4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

Commit message: Updating schematic with Oshpark/Digikey order
Updates to add various components and capability.

2.2 Basic Sensor Suite
Parts:
- removed D3: D, Diode_THT:D_T-1_P5.08mm_Horizontal, symbol Device:D
- added D3: D_Bridge_+AA-, TTS-UART:KBP306GTB, symbol Device:D_Bridge_+AA-
- added R2: 4.7k, Resistor_THT:R_Axial_DIN0204_L3.6mm_D1.6mm_P5.08mm_Horizontal, symbol Device:R
- D1, D2: footprint TTS-UART:DO204-10 -> Diode_SMD:D_SOD-923
Connections:
- wire segments 100 -> 116
Other:
- moved on the sheet: D4
Changed lines of the file:
@@
 F 0 "D1" V 2254 1530 50  0000 L CNN
 F 1 "D_Zener" V 2345 1530 50  0000 L CNN
-F 2 "TTS-UART:DO204-10" H 2300 1450 50  0001 C CNN
+F 2 "Diode_SMD:D_SOD-923" H 2300 1450 50  0001 C CNN
 F 3 "~" H 2300 1450 50  0001 C CNN
 	1    2300 1450
@@
 F 0 "D2" V 2554 2630 50  0000 L CNN
 F 1 "D_Zener" V 2645 2630 50  0000 L CNN
-F 2 "TTS-UART:DO204-10" H 2600 2550 50  0001 C CNN
+F 2 "Diode_SMD:D_SOD-923" H 2600 2550 50  0001 C CNN
 F 3 "~" H 2600 2550 50  0001 C CNN
 	1    2600 2550
@@
 Wire Wire Line
 	2600 2700 2600 2750
-$Comp
-L power:GND #PWR01
-U 1 1 5F8F4209
-P 1250 2350
-F 0 "#PWR01" H 1250 2100 50  0001 C CNN
-F 1 "GND" H 1255 2177 50  0000 C CNN
-F 2 "" H 1250 2350 50  0001 C CNN
-F 3 "" H 1250 2350 50  0001 C CNN
-	1    1250 2350
-	1    0    0    -1
-$EndComp
 Wire Wire Line
 	1250 2300 1250 2350
@@
 Wire Wire Line
 	2150 6150 2150 5850
-Connection ~ 2150 5850
-Wire Wire Line
-	2150 5850 3250 5850
-$Comp
-L Device:D D3
-U 1 1 5F8FD3DE
-P 3400 5850
-F 0 "D3" V 3354 5930 50  0000 L CNN
-F 1 "D" V 3445 5930 50  0000 L CNN
-F 2 "Diode_THT:D_T-1_P5.08mm_Horizontal" H 3400 5850 50  0001 C CNN
-F 3 "~" H 3400 5850 50  0001 C CNN
-	1    3400 5850
-	-1   0    0    1
-$EndComp
-Wire Wire Line
-	3550 5850 4350 5850
-$Comp
-L power:GND #PWR05
-U 1 1 5F90012A
-P 1750 6250
-F 0 "#PWR05" H 1750 6000 50  0001 C CNN
-F 1 "GND" H 1755 6077 50  0000 C CNN
-F 2 "" H 1750 6250 50  0001 C CNN
-F 3 "" H 1750 6250 50  0001 C CNN
-	1    1750 6250
-	1    0    0    -1
-$EndComp
 Wire Wire Line
 	2050 6150 2050 6000
-Wire Wire Line
-	2050 6000 1750 6000
-Wire Wire Line
-	1750 6000 1750 6250
 Text Label 6950 2350 0    50   ~ 0
 D10
@@
 U 1 1 5F8FB33C
 P 2150 6350
-F 0 "J5" V 2022 6430 50  0000 L CNN
-F 1 "Screw_Terminal_01x02" V 2113 6430 50  0000 L CNN
+F 0 "J5" V 2150 6450 50  0000 L CNN
+F 1 "Screw_Terminal_01x02" V 2250 6050 50  0000 L CNN
 F 2 "TerminalBlock_Phoenix:TerminalBlock_Phoenix_PT-1,5-2-5.0-H_1x02_P5.00mm_Horizontal" H 2150 6350 50  0001 C CNN
 F 3 "~" H 2150 6350 50  0001 C CNN
@@
 	0    1    1    0
 $EndComp
-$Comp
-L power:GND #PWR02
-U 1 1 5F913976
-P 1250 3400
-F 0 "#PWR02" H 1250 3150 50  0001 C CNN
-F 1 "GND" H 1255 3227 50  0000 C CNN
-F 2 "" H 1250 3400 50  0001 C CNN
-F 3 "" H 1250 3400 50  0001 C CNN
-	1    1250 3400
-	1    0    0    -1
-$EndComp
 Wire Wire Line
 	1250 3350 1250 3400
-$Comp
-L power:GND #PWR03
-U 1 1 5F918C16
-P 1250 4450
-F 0 "#PWR03" H 1250 4200 50  0001 C CNN
-F 1 "GND" H 1255 4277 50  0000 C CNN
-F 2 "" H 1250 4450 50  0001 C CNN
-F 3 "" H 1250 4450 50  0001 C CNN
-	1    1250 4450
-	1    0    0    -1
-$EndComp
 Wire Wire Line
 	1250 4450 1250 4400
@@
 Wire Wire Line
 	850  4750 850  5850
-$Comp
-L power:GND #PWR04
-U 1 1 5F9418F0
-P 1250 5500
-F 0 "#PWR04" H 1250 5250 50  0001 C CNN
-F 1 "GND" H 1255 5327 50  0000 C CNN
-F 2 "" H 1250 5500 50  0001 C CNN
-F 3 "" H 1250 5500 50  0001 C CNN
-	1    1250 5500
-	1    0    0    -1
-$EndComp
-Wire Wire Line
-	1250 5500 1250 5450
 Wire Wire Line
 	2000 3700 2000 4750
@@
 L Device:LED D4
 U 1 1 5F920F36
+P 7350 4900
+F 0 "D4" V 7389 4782 50  0000 R CNN
+F 1 "RED" V 7298 4782 50  0000 R CNN
+F 2 "digikey-kicad-library:LED_3mm_Radial" H 7350 4900 50  0001 C CNN
+F 3 "~" H 7350 4900 50  0001 C CNN
+	1    7350 4900
+	0    -1   -1   0
+$EndComp
+Wire Wire Line
+	6950 4350 7350 4350
+Wire Wire Line
+	7350 4350 7350 4400
+Wire Wire Line
+	7350 5100 7350 5050
+$Comp
+L Device:D_Bridge_+AA- D3
+U 1 1 5F9B1CA7
+P 3200 5650
+F 0 "D3" H 3150 5650 50  0000 L CNN
+F 1 "D_Bridge_+AA-" H 3300 5850 50  0000 L CNN
+F 2 "TTS-UART:KBP306GTB" H 3200 5650 50  0001 C CNN
+F 3 "~" H 3200 5650 50  0001 C CNN
+	1    3200 5650
+	1    0    0    -1
+$EndComp
+Wire Wire Line
+	2150 5850 2550 5850
+Wire Wire Line
+	2550 5850 2550 5300
+Wire Wire Line
+	2550 5300 3200 5300
+Wire Wire Line
+	3200 5300 3200 5350
+Connection ~ 2150 5850
+$Comp
+L power:GND #PWR01
+U 1 1 5F9CBB76
+P 2850 5700
+F 0 "#PWR01" H 2850 5450 50  0001 C CNN
+F 1 "GND" H 2855 5527 50  0000 C CNN
+F 2 "" H 2850 5700 50  0001 C CNN
+F 3 "" H 2850 5700 50  0001 C CNN
+	1    2850 5700
+	1    0    0    -1
+$EndComp
+Wire Wire Line
+	2900 5650 2850 5650
+Wire Wire Line
+	2850 5650 2850 5700
+Wire Wire Line
+	1250 4450 1000 4450
+Wire Wire Line
+	1000 4450 1000 5450
+Wire Wire Line
+	1250 5450 1000 5450
+Connection ~ 1000 5450
+Wire Wire Line
+	1000 5450 1000 6000
+Wire Wire Line
+	1000 4450 1000 3400
+Wire Wire Line
+	1000 3400 1250 3400
+Connection ~ 1000 4450
+Wire Wire Line
+	1000 3400 1000 2350
+Wire Wire Line
+	1000 2350 1250 2350
+Connection ~ 1000 3400
+Wire Wire Line
+	1000 6000 2050 6000
+Wire Wire Line
+	2050 6000 3200 6000
+Wire Wire Line
+	3200 6000 3200 5950
+Connection ~ 2050 6000
+Wire Wire Line
+	3500 5650 3550 5650
+Wire Wire Line
+	3550 5650 3550 5850
+Wire Wire Line
+	3550 5850 4350 5850
+$Comp
+L power:VCC #PWR02
+U 1 1 5FA4D1B3
+P 7350 5100
+F 0 "#PWR02" H 7350 4950 50  0001 C CNN
+F 1 "VCC" H 7365 5273 50  0000 C CNN
+F 2 "" H 7350 5100 50  0001 C CNN
+F 3 "" H 7350 5100 50  0001 C CNN
+	1    7350 5100
+	-1   0    0    1
+$EndComp
+$Comp
+L Device:R R2
+U 1 1 5FA529EF
 P 7350 4550
-F 0 "D4" V 7389 4432 50  0000 R CNN
-F 1 "RED" V 7298 4432 50  0000 R CNN
-F 2 "digikey-kicad-library:LED_3mm_Radial" H 7350 4550 50  0001 C CNN
+F 0 "R2" H 7420 4596 50  0000 L CNN
+F 1 "4.7k" H 7420 4505 50  0000 L CNN
+F 2 "Resistor_THT:R_Axial_DIN0204_L3.6mm_D1.6mm_P5.08mm_Horizontal" V 7280 4550 50  0001 C CNN
 F 3 "~" H 7350 4550 50  0001 C CNN
 	1    7350 4550
-	0    -1   -1   0
-$EndComp
-Wire Wire Line
-	6950 4350 7350 4350
-Wire Wire Line
-	7350 4350 7350 4400
-$Comp
-L power:GND #PWR0101
-U 1 1 5F925787
-P 7350 4750
-F 0 "#PWR0101" H 7350 4500 50  0001 C CNN
-F 1 "GND" H 7355 4577 50  0000 C CNN
-F 2 "" H 7350 4750 50  0001 C CNN
-F 3 "" H 7350 4750 50  0001 C CNN
-	1    7350 4750
-	1    0    0    -1
-$EndComp
-Wire Wire Line
-	7350 4750 7350 4700
+	1    0    0    -1
+$EndComp
+Wire Wire Line
+	7350 4700 7350 4750
 $EndSCHEMATC
